File: hardware/slackdsp_mini.kicad_pcb (KiCad board)
At the start: 2 copper layers, 48.3 x 55.9 mm, 48 parts, among them K1 UART, P1 DC In, P2 In, P3 Out, P4 LED, P5 ICSP, Q1 JFET_N, U1 DSPIC33FJ128GP804, U2 WM8510, U3 7833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

Commit message: Updated PCB
Parts:
- C1, C11, C5, C6, C7, C8, C9: footprint SM1210L -> Capacitors_SMD:C_1210_HandSoldering
- C10: footprint C1V5 -> Capacitors_THT:CP_Radial_D5.0mm_P2.50mm
- C12, C13, C14, C15, C2, C3, C4: footprint SM1206 -> Capacitors_SMD:C_1206
- D1, D2: footprint SM1812 -> Capacitors_SMD:C_1812
- D3: footprint LED-3MM -> LEDs:LED_D3.0mm
- K1: footprint SIL-3 -> Pin_Headers:Pin_Header_Straight_1x03_Pitch2.54mm
- P1, P2, P3, P4: footprint SIL-2 -> Pin_Headers:Pin_Header_Straight_1x02_Pitch2.54mm
- P5: footprint SIL-5 -> Pin_Headers:Pin_Header_Straight_1x05_Pitch2.54mm
- Q1: footprint SOT23 -> TO_SOT_Packages_SMD:SOT-23
- R1, R10, R11, R12, R13, R14, R15, R16, R2, R3, R4, R5, R6, R8, R9: footprint SM1206 -> Resistors_SMD:R_1206
- R7: value 10k -> 3k3; footprint SM1206 -> Resistors_SMD:R_1206
- RV1, RV2, RV3: footprint POT_16mm -> slacklib:POT_16mm
- U1: footprint TQFP44 -> Housings_QFP:TQFP-44_10x10mm_Pitch0.8mm
- U2: footprint SSOP28 -> Housings_SSOP:SSOP-28_5.3x10.2mm_Pitch0.65mm
- U3: footprint SOT223 -> TO_SOT_Packages_SMD:SOT-223
- U4: footprint SO8-Narrow -> slacklib:SO8-Narrow
- moved P5 6.22 mm to (47.6, 64.1), turned to 270 degrees
- moved K1 2.62 mm to (66.0, 76.2), turned to 180 degrees
- moved C10 1.37 mm to (30.5, 59.7)
- moved P3 1.27 mm to (24.1, 31.1), turned to 90 degrees
- moved D3 1.27 mm to (44.5, 74.9)
- moved P1 1.27 mm to (40.6, 76.2), turned to 180 degrees
- moved P2 1.27 mm to (67.3, 31.1), turned to 270 degrees
- moved P4 1.27 mm to (50.8, 76.2), turned to 180 degrees
- moved C9 0.80 mm to (30.5, 45.7)
- moved C7 0.80 mm to (25.4, 45.7)
- moved R11 0.63 mm to (61.0, 73.0)
- turned Q1 to 90 degrees
- turned U2 to 0 degrees
- turned U3 to 270 degrees
Connections:
- P5 pad 2: (no net) -> Net-(P5-Pad2)
- U1 pad 12: (no net) -> Net-(U1-Pad12)
- U1 pad 13: (no net) -> Net-(U1-Pad13)
- U1 pad 15: (no net) -> Net-(U1-Pad15)
- U1 pad 19: (no net) -> Net-(U1-Pad19)
- U1 pad 20: (no net) -> Net-(U1-Pad20)
- U1 pad 26: (no net) -> Net-(U1-Pad26)
- U1 pad 27: (no net) -> Net-(U1-Pad27)
- U1 pad 30: (no net) -> Net-(U1-Pad30)
- U1 pad 31: (no net) -> Net-(U1-Pad31)
- U1 pad 34: (no net) -> Net-(U1-Pad34)
- U1 pad 35: (no net) -> Net-(U1-Pad35)
- U1 pad 38: (no net) -> Net-(U1-Pad38)
- U1 pad 41: (no net) -> Net-(U1-Pad41)
- U1 pad 42: (no net) -> Net-(U1-Pad42)
- U1 pad 43: (no net) -> Net-(U1-Pad43)
- U1 pad 44: (no net) -> Net-(U1-Pad44)
- U1 pad 8: (no net) -> Net-(U1-Pad8)
- U2 pad 2: (no net) -> Net-(U2-Pad2)
- U2 pad 22: (no net) -> Net-(U2-Pad22)
- U2 pad 25: (no net) -> Net-(U2-Pad25)
- U2 pad 3: (no net) -> Net-(U2-Pad3)
- U2 pad 4: (no net) -> Net-(U2-Pad4)
- U2 pad 5: (no net) -> Net-(U2-Pad5)
Routing:
- net GND: track 357.7 -> 343.1 mm
- net POT2: track 21.8 -> 26.3 mm
- net MONOOUT: track 25.9 -> 28.4 mm
- net VCC: track 260.4 -> 262.6 mm
- net +9V: track 53.0 -> 54.6 mm, vias 2 -> 1
- net Net-(K1-Pad2): track 3.69 -> 5.16 mm
- net Net-(C9-Pad1): track 5.73 -> 6.97 mm
- net Net-(R12-Pad1): track 4.97 -> 3.77 mm
- net CLOCK: track 34.4 -> 35.5 mm
- net MIC2: track 4.33 -> 5.24 mm
Other:
- board text added: "v1.1 08072017"
- board text removed: "v1.0 18112014"
