File: hardware/slackdsp_mini.sch (KiCad schematic (older format))
At the start: 48 parts, among them K1 UART, P1 DC In, P2 In, P3 Out, P4 LED, P5 ICSP, Q1 JFET_N, U1 DSPIC33FJ128GP804, U2 WM8510, U3 7833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

Commit message: Updated PCB
Parts:
- C1, C11, C5, C6, C7, C8, C9: footprint ~ -> Capacitors_SMD:C_1210_HandSoldering
- C10: footprint ~ -> Capacitors_THT:CP_Radial_D5.0mm_P2.50mm
- C12, C13, C14, C15, C2, C3, C4: footprint ~ -> Capacitors_SMD:C_1206
- D1, D2: footprint ~ -> Capacitors_SMD:C_1812
- D3: footprint ~ -> LEDs:LED_D3.0mm
- K1: footprint (none) -> Pin_Headers:Pin_Header_Straight_1x03_Pitch2.54mm
- P1, P2, P3, P4: footprint (none) -> Pin_Headers:Pin_Header_Straight_1x02_Pitch2.54mm
- P5: footprint (none) -> Pin_Headers:Pin_Header_Straight_1x05_Pitch2.54mm
- Q1: footprint ~ -> TO_SOT_Packages_SMD:SOT-23
- R1, R10, R11, R12, R13, R14, R15, R16, R2, R3, R4, R5, R6, R7, R8, R9: footprint ~ -> Resistors_SMD:R_1206
- RV1, RV2, RV3: footprint ~ -> slacklib:POT_16mm
- U1: footprint ~ -> Housings_QFP:TQFP-44_10x10mm_Pitch0.8mm
- U2: footprint ~ -> Housings_SSOP:SSOP-28_5.3x10.2mm_Pitch0.65mm
- U3: footprint ~ -> TO_SOT_Packages_SMD:SOT-223
- U4: footprint (none) -> slacklib:SO8-Narrow
Other:
- moved on the sheet: C10
